File: t41_2_power_amplifier.kicad_pcb (KiCad board)
At the start: 2 copper layers, 100 x 100 mm, 59 parts, among them J1 5-1814832-1, J2 5-1814832-1, J3 B2B-XH-A_LF__SN_, J5 Screw_Terminal_01x02, Q1 Q_NMOS_GSD, Q2 Q_NPN_BCE, Q3 Q_NMOS_GSD, Q4 Q_NPN_BCE, Q5 Q_PMOS_GSD, Q6 Q_NPN_BEC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

Commit message: Beefed up main supply trace to final.
Parts:
- moved E1 1.25 mm to (166.8, 109.8)
Routing:
- net GND: track 12.7 -> 9.65 mm
- net /12V_OUT_FIL: track 36.8 -> 38.7 mm, vias 2 -> 3
- net Net-(U1-VIN): track 83.6 -> 84.1 mm
Changed lines of the file:
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@@
 	(footprint "28F0121_0SR_10:FB_28F0121-0SR-10"
 		(layer "F.Cu")
-		(at 165.55 109.85 90)
+		(at 166.8 109.85 90)
 		(property "Reference" "E1"
 			(at 0 2.95 180)
@@
 		)
 		(property "Value" "Q_NMOS_GSD"
-			(at 0 -8 270)
+			(at 0 -8 -90)
 			(unlocked yes)
 			(layer "F.Fab")
@@
 		)
 		(fp_text user "${REFERENCE}"
-			(at 0 -6.5 270)
+			(at 0 -6.5 -90)
 			(unlocked yes)
 			(layer "F.Fab")
@@
 		(tags "resistor")
 		(property "Reference" "R2"
-			(at 0 -1.82 360)
+			(at 0 -1.82 0)
 			(layer "F.SilkS")
 			(effects
@@
 		)
 		(fp_text user "${REFERENCE}"
-			(at 0 0 360)
+			(at 0 0 0)
 			(layer "F.Fab")
 			(effects
@@
 	(segment
 		(start 164.8 90)
-		(end 165.55 90)
-		(width 1)
+		(end 166 90)
+		(width 1.5)
 		(layer "F.Cu")
 		(net 1)
 	)
 	(segment
-		(start 165.55 108.06)
-		(end 165.55 90)
-		(width 1)
+		(start 164.8 90)
+		(end 163.65 90)
+		(width 1.5)
 		(layer "F.Cu")
 		(net 1)
 	)
 	(segment
-		(start 164.8 90)
-		(end 163.65 90)
-		(width 1)
+		(start 166.8 108.06)
+		(end 166.8 90.8)
+		(width 2)
+		(layer "F.Cu")
+		(net 1)
+	)
+	(segment
+		(start 166.8 90.8)
+		(end 166 90)
+		(width 2)
 		(layer "F.Cu")
 		(net 1)
@@
 	)
 	(via
+		(at 166 90)
+		(size 1)
+		(drill 0.5)
+		(layers "F.Cu" "B.Cu")
+		(net 1)
+	)
+	(via
 		(at 164.8 90)
 		(size 1)
@@
 		(start 163.65 90)
 		(end 164.8 90)
-		(width 1)
+		(width 1.5)
 		(layer "B.Cu")
 		(net 1)
@@
 		(start 154.25 90)
 		(end 163.65 90)
-		(width 1)
+		(width 1.5)
+		(layer "B.Cu")
+		(net 1)
+	)
+	(segment
+		(start 164.8 90)
+		(end 166 90)
+		(width 1.5)
 		(layer "B.Cu")
 		(net 1)
@@
 		(start 151 90)
 		(end 154.25 90)
-		(width 1)
+		(width 1.5)
 		(layer "B.Cu")
 		(net 1)
@@
 		(start 156.5 79.9)
 		(end 156.5 81.7)
-		(width 1)
+		(width 1.5)
 		(layer "F.Cu")
 		(net 2)
 	)
 	(segment
-		(start 156.5 79.9)
-		(end 155.7 80.7)
-		(width 0.2)
+		(start 157.8 98.8)
+		(end 157.8 99.1)
+		(width 0.25)
 		(layer "F.Cu")
 		(net 2)
@@
 	)
 	(segment
-		(start 156.6 79.9)
-		(end 157.7 81)
-		(width 0.2)
-		(layer "F.Cu")
-		(net 2)
-	)
-	(segment
-		(start 155.7 80.7)
-		(end 155.2 81.2)
-		(width 0.2)
-		(layer "F.Cu")
-		(net 2)
-	)
-	(segment
 		(start 156.5 100.4)
 		(end 156.5 99)
-		(width 1)
+		(width 1.5)
 		(layer "F.Cu")
 		(net 2)
@@
 	)
 	(via
-		(at 167.25 125.55)
+		(at 167.75 125.75)
 		(size 1)
 		(drill 0.5)
@@
 	)
 	(via
-		(at 163.7 91.7)
+		(at 164.15 92)
 		(size 1)
 		(drill 0.5)
@@
 	)
 	(via
-		(at 148.6 124.8)
+		(at 148.95 124.2)
 		(size 1)
 		(drill 0.5)
@@
 	)
 	(via
-		(at 136.25 129.5)
+		(at 136.25 130.25)
 		(size 1)
 		(drill 0.5)
@@
 	)
 	(via
-		(at 144.9 125.75)
+		(at 144.7 125.05)
 		(size 1)
 		(drill 0.5)
@@
 	)
 	(via
-		(at 163.5 88.3)
+		(at 163.85 87.9)
 		(size 1)
 		(drill 0.5)
@@
 	)
 	(via
-		(at 163.05 126)
+		(at 162.75 125.75)
 		(size 1)
 		(drill 0.5)
@@
 	)
 	(segment
+		(start 158.8 127.85)
+		(end 158.8 126.8)
+		(width 0.5)
+		(layer "F.Cu")
+		(net 11)
+	)
+	(segment
 		(start 129.275 120.925)
 		(end 120.7 112.35)
@@
 	)
 	(segment
-		(start 132.675 120.95)
-		(end 132.7 120.925)
-		(width 0.25)
+		(start 165.15 120)
+		(end 166.8 118.35)
+		(width 2)
 		(layer "F.Cu")
 		(net 11)
 	)
 	(segment
-		(start 147.95 126.3)
-		(end 145.35 123.7)
-		(width 0.5)
+		(start 132.675 120.95)
+		(end 132.7 120.925)
+		(width 0.25)
 		(layer "F.Cu")
 		(net 11)
 	)
 	(segment
-		(start 165.55 127.45)
-		(end 165.15 127.85)
-		(width 1)
+		(start 157.725 125.725)
+		(end 147.375 125.725)
+		(width 0.5)
 		(layer "F.Cu")
 		(net 11)
@@
 		(start 165.15 127.85)
 		(end 173.1 127.85)
-		(width 1)
-		(layer "F.Cu")
-		(net 11)
-	)
-	(segment
-		(start 158.8 126.8)
-		(end 158.3 126.3)
-		(width 0.5)
+		(width 1.5)
 		(layer "F.Cu")
 		(net 11)
@@
 		(start 158.8 127.85)
 		(end 165.15 127.85)
-		(width 1)
+		(width 1.5)
 		(layer "F.Cu")
 		(net 11)
 	)
 	(segment
-		(start 158.8 127.85)
-		(end 158.8 126.8)
-		(width 0.5)
+		(start 132.7 120.925)
+		(end 129.275 120.925)
+		(width 0.25)
 		(layer "F.Cu")
 		(net 11)
 	)
 	(segment
-		(start 158.3 126.3)
-		(end 147.95 126.3)
+		(start 145.35 123.7)
+		(end 132.7 123.7)
 		(width 0.5)
 		(layer "F.Cu")
@@
 	)
 	(segment
-		(start 165.55 111.64)
-		(end 165.55 127.45)
-		(width 1)
+		(start 166.8 118.35)
+		(end 166.8 111.64)
+		(width 2)
 		(layer "F.Cu")
 		(net 11)
 	)
 	(segment
-		(start 132.7 120.925)
-		(end 129.275 120.925)
-		(width 0.25)
+		(start 158.8 126.8)
+		(end 157.725 125.725)
+		(width 0.5)
 		(layer "F.Cu")
 		(net 11)
 	)
 	(segment
-		(start 145.35 123.7)
-		(end 132.7 123.7)
+		(start 158.8 127.85)
+		(end 158.8 131.15)
 		(width 0.5)
 		(layer "F.Cu")
@@
 	)
 	(segment
-		(start 158.8 127.85)
-		(end 158.8 131.15)
+		(start 147.375 125.725)
+		(end 145.35 123.7)
 		(width 0.5)
 		(layer "F.Cu")
@@
 	)
 	(segment
+		(start 165.15 127.85)
+		(end 165.15 120)
+		(width 2)
+		(layer "F.Cu")
+		(net 11)
+	)
+	(segment
 		(start 115.7 116.5)
 		(end 115.7 113.2)
@@
 		(start 150.75 127.85)
 		(end 155.22 127.85)
-		(width 1)
+		(width 1.5)
 		(layer "F.Cu")
 		(net 13)
@@
 		(start 131.46 127.8)
 		(end 140.85 127.8)
-		(width 1)
+		(width 2.5)
 		(layer "F.Cu")
 		(net 20)
@@
 		(start 140.9 127.85)
 		(end 147.17 127.85)
-		(width 1)
+		(width 1.5)
 		(layer "F.Cu")
 		(net 20)
@@
 		(start 107.05 127.8)
 		(end 118 127.8)
-		(width 1)
+		(width 2.5)
 		(layer "F.Cu")
 		(net 23)

Commit message: Added another stage to the input.
Parts:
- added H1: MountingHole_Pad, MountingHole:MountingHole_4.3mm_M4_DIN965_Pad, F.Cu at (105.0, 55.0)
- added H2: MountingHole_Pad, MountingHole:MountingHole_4.3mm_M4_DIN965_Pad, F.Cu at (105.0, 145.0)
- added H3: MountingHole_Pad, MountingHole:MountingHole_4.3mm_M4_DIN965_Pad, F.Cu at (195.0, 145.0)
- added H4: MountingHole_Pad, MountingHole:MountingHole_4.3mm_M4_DIN965_Pad, F.Cu at (195.0, 55.0)
- moved R12 15.4 mm to (108.9, 85.8), turned to 0 degrees
- moved R10 14.3 mm to (121.0, 84.7), turned to 180 degrees
- moved Q4 13.5 mm to (113.5, 91.5)
- moved C15 13.5 mm to (115.5, 80.0)
- moved Q2 13.5 mm to (115.4, 85.1)
- moved R9 13.5 mm to (119.6, 88.7)
- moved C16 12.3 mm to (121.1, 93.0), turned to 180 degrees
- moved R13 11.8 mm to (107.0, 90.0), turned to -90 degrees
- moved L1 11.7 mm to (116.7, 98.0)
- moved R14 11.7 mm to (120.3, 98.0)
- moved C17 11.4 mm to (121.6, 102.3)
- moved Q5 8.84 mm to (116.7, 103.5)
- moved R19 8.84 mm to (116.6, 107.5)
- moved Q6 8.16 mm to (112.0, 108.7)
- moved R20 6.31 mm to (112.5, 112.6), turned to 0 degrees
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Connections:
- C16 pad 1: Net-(T3-AA) -> Net-(T3-AB)
- T3 pad 1: Net-(T3-AA) -> GND
- T3 pad 2: GND -> Net-(T3-AB)
Routing:
- net Net-(U1-VIN): track 84.1 -> 70.3 mm
- net Net-(J2-Pad2): track 9.61 -> 0.00 mm
- net Net-(C15-Pad2): track 5.56 -> 0.02 mm
- net /TXRX: track 33.9 -> 29.0 mm
- net Net-(T3-AB): track 0.00 -> 4.65 mm
- net Net-(Q5-S): track 10.4 -> 6.00 mm
- net Net-(T3-AA): track 3.22 -> 0.00 mm
- net Net-(Q2-B): track 8.97 -> 5.82 mm
- net Net-(Q5-G): track 5.82 -> 3.15 mm
- net Net-(Q6-B): track 2.45 -> 0.00 mm
- net Net-(Q2-C): track 23.3 -> 24.0 mm
- net GND: vias 83 -> 79
Other:
- outline, holes or cut-outs redrawn

Commit message: Release V1.0.
Parts:
- added C19: 0.1uF, Capacitor_SMD:C_1206_3216Metric, F.Cu at (116.4, 66.2)
- added C21: 0.1uF, Capacitor_SMD:C_1206_3216Metric, F.Cu at (123.2, 78.3)
- added Q7: Q_NPN_BEC, Package_TO_SOT_SMD:SOT-23-3, F.Cu at (121.7, 67.2)
- added Q8: Q_NPN_BEC, Package_TO_SOT_SMD:SOT-23-3, F.Cu at (121.8, 71.3)
- added R21: 150, Resistor_SMD:R_1206_3216Metric, F.Cu at (117.8, 70.5)
- added R22: 1000, Resistor_SMD:R_1206_3216Metric, F.Cu at (123.2, 75.2)
- added R23: 10, Resistor_SMD:R_1206_3216Metric, F.Cu at (125.4, 71.0)
- added R3: 1000, Resistor_SMD:R_1206_3216Metric, F.Cu at (122.0, 63.5)
- added R4: 1500, Resistor_SMD:R_1206_3216Metric, F.Cu at (116.7, 63.0)
- R10: value 56 -> 1500
- R12: value 56 -> 150
- R13: value 56 -> 10
- R9: value 56 -> 1000
- moved R15 8.44 mm to (114.9, 73.4), turned to 90 degrees
- moved R16 5.59 mm to (112.0, 73.4), turned to 90 degrees
- moved C17 4.67 mm to (123.4, 98.0), turned to 90 degrees
- moved R18 3.42 mm to (113.4, 69.3)
- moved C15 3.41 mm to (118.5, 78.3), turned to 90 degrees
Connections:
- C15 pad 2: Net-(C15-Pad2) -> Net-(Q7-C)
- R15 pad 2: Net-(C15-Pad2) -> Net-(C19-Pad2)
- R18 pad 2: Net-(C15-Pad2) -> Net-(C19-Pad2)
Routing:
- net /12V_IN_FIL: track 10.0 -> 40.2 mm
- net Net-(Q7-C): track 0.00 -> 16.5 mm
- net Net-(U1-VIN): track 70.3 -> 82.6 mm
- net Net-(J2-Pad2): track 0.00 -> 8.63 mm
- net Net-(Q7-B): track 0.00 -> 8.07 mm
- net Net-(Q7-E): track 0.00 -> 7.57 mm
- net Net-(C19-Pad2): track 0.00 -> 5.71 mm
- net /TXRX: track 29.0 -> 34.0 mm
- net Net-(Q2-B): track 5.82 -> 9.77 mm
- net Net-(Q5-G): track 3.15 -> 6.29 mm
- net Net-(Q6-B): track 0.00 -> 2.77 mm
- net Net-(Q8-E): track 0.00 -> 2.65 mm
- net GND: vias 79 -> 133
