File: t41_2_power_amplifier.kicad_sch (KiCad schematic)
At the start: 72 parts, among them J1 5-1814832-1, J2 5-1814832-1, J3 B2B-XH-A_LF__SN_, J5 Screw_Terminal_01x02, Q1 Q_NMOS_GSD, Q2 Q_NPN_BCE, Q3 Q_NMOS_GSD, Q4 Q_NPN_BCE, Q5 Q_PMOS_GSD, Q6 Q_NPN_BEC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

Commit message: Release V1.0.
Parts:
- removed Q7, Q8: Q_NPN_BCE, Package_TO_SOT_SMD:SOT-23-3, symbol Device:Q_NPN_BCE
- added Q7, Q8: Q_NPN_BEC, Package_TO_SOT_SMD:SOT-23-3, symbol Device:Q_NPN_BEC
- R10, R4: value 56 -> 1500
- R12, R21: value 56 -> 150
- R13, R23: value 56 -> 10
- R3, R9: value 56 -> 1000
Connections:
- net at R23.2: now also Q8.2 (E)
- net at R21.2: now also Q7.2 (E), Q8.1 (B)
- net at C15.2, R22.1, R3.2: now also Q7.3 (C), Q8.3 (C)
- net at C19.1, R3.1, R4.2: now also Q7.1 (B)
Changed lines of the file:
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@@
 	)
 	(symbol
+		(lib_id "Device:Q_NPN_BEC")
+		(at 54.61 63.5 0)
+		(unit 1)
+		(exclude_from_sim no)
+		(in_bom yes)
+		(on_board yes)
+		(dnp no)
+		(fields_autoplaced yes)
+		(property "Reference" "Q7"
+			(at 59.69 62.2299 0)
+			(effects
+				(font
+					(size 1.27 1.27)
+				)
+				(justify left)
+			)
+		)
+		(property "Value" "Q_NPN_BEC"
+			(at 59.69 64.7699 0)
+			(effects
+				(font
+					(size 1.27 1.27)
+				)
+				(justify left)
+			)
+		)
+		(property "Footprint" "Package_TO_SOT_SMD:SOT-23-3"
+			(at 59.69 60.96 0)
+			(effects
+				(font
+					(size 1.27 1.27)
+				)
+				(hide yes)
+			)
+		)
+		(property "Datasheet" "~"
+			(at 54.61 63.5 0)
+			(effects
+				(font
+					(size 1.27 1.27)
+				)
+				(hide yes)
+			)
+		)
+		(property "Description" "NPN transistor, base/emitter/collector"
+			(at 54.61 63.5 0)
+			(effects
+				(font
+					(size 1.27 1.27)
+				)
+				(hide yes)
+			)
+		)
+		(pin "3"
+		)
+		(pin "1"
+		)
+		(pin "2"
+		)
+		(instances
+			(project ""
+				(path "/2dfc3106-0fe9-4b2c-b32a-a54bf0a73e15"
+					(reference "Q7")
+					(unit 1)
+				)
+			)
+		)
+	)
+	(symbol
 		(lib_id "Auto_Fuse_Holder:3587TR")
 		(at 41.91 144.78 0)
@@
 			)
 		)
-		(property "Value" "56"
+		(property "Value" "10"
 			(at 71.12 73.66 90)
 			(effects
@@
 			)
 		)
-		(property "Value" "56"
+		(property "Value" "150"
 			(at 54.61 73.66 90)
 			(effects
@@
 	)
 	(symbol
-		(lib_id "Device:Q_NPN_BCE")
-		(at 54.61 63.5 0)
-		(unit 1)
-		(exclude_from_sim no)
-		(in_bom yes)
-		(on_board yes)
-		(dnp no)
-		(property "Reference" "Q7"
-			(at 48.26 48.26 0)
-			(effects
-				(font
-					(size 1.27 1.27)
-				)
-				(justify left)
-			)
-		)
-		(property "Value" "Q_NPN_BCE"
-			(at 52.07 48.26 0)
-			(effects
-				(font
-					(size 1.27 1.27)
-				)
-				(justify left)
-			)
-		)
-		(property "Footprint" "Package_TO_SOT_SMD:SOT-23-3"
-			(at 59.69 60.96 0)
-			(effects
-				(font
-					(size 1.27 1.27)
-				)
-				(hide yes)
-			)
-		)
-		(property "Datasheet" "~"
-			(at 54.61 63.5 0)
-			(effects
-				(font
-					(size 1.27 1.27)
-				)
-				(hide yes)
-			)
-		)
-		(property "Description" "NPN transistor, base/collector/emitter"
-			(at 54.61 63.5 0)
-			(effects
-				(font
-					(size 1.27 1.27)
-				)
-				(hide yes)
-			)
-		)
-		(pin "1"
-		)
-		(pin "2"
-		)
-		(pin "3"
-		)
-		(instances
-			(project "t41_2_power_amplifier"
-				(path "/2dfc3106-0fe9-4b2c-b32a-a54bf0a73e15"
-					(reference "Q7")
-					(unit 1)
-				)
-			)
-		)
-	)
-	(symbol
 		(lib_id "power:GND")
 		(at 213.36 120.65 0)
@@
 			)
 		)
-		(property "Value" "56"
+		(property "Value" "1000"
 			(at 90.17 53.34 90)
 			(effects
@@
 			)
 		)
-		(property "Value" "56"
+		(property "Value" "1500"
 			(at 90.17 73.66 90)
 			(effects
@@
 			)
 		)
-		(property "Value" "56"
+		(property "Value" "1500"
 			(at 45.72 73.66 90)
 			(effects
@@
 	)
 	(symbol
-		(lib_id "Device:Q_NPN_BCE")
-		(at 71.12 63.5 0)
-		(unit 1)
-		(exclude_from_sim no)
-		(in_bom yes)
-		(on_board yes)
-		(dnp no)
-		(property "Reference" "Q8"
-			(at 67.31 54.61 0)
-			(effects
-				(font
-					(size 1.27 1.27)
-				)
-				(justify left)
-			)
-		)
-		(property "Value" "Q_NPN_BCE"
-			(at 60.96 57.15 0)
-			(effects
-				(font
-					(size 1.27 1.27)
-				)
-				(justify left)
-			)
-		)
-		(property "Footprint" "Package_TO_SOT_SMD:SOT-23-3"
-			(at 76.2 60.96 0)
-			(effects
-				(font
-					(size 1.27 1.27)
-				)
-				(hide yes)
-			)
-		)
-		(property "Datasheet" "~"
-			(at 71.12 63.5 0)
-			(effects
-				(font
-					(size 1.27 1.27)
-				)
-				(hide yes)
-			)
-		)
-		(property "Description" "NPN transistor, base/collector/emitter"
-			(at 71.12 63.5 0)
-			(effects
-				(font
-					(size 1.27 1.27)
-				)
-				(hide yes)
-			)
-		)
-		(pin "1"
-		)
-		(pin "2"
-		)
-		(pin "3"
-		)
-		(instances
-			(project "t41_2_power_amplifier"
-				(path "/2dfc3106-0fe9-4b2c-b32a-a54bf0a73e15"
-					(reference "Q8")
-					(unit 1)
-				)
-			)
-		)
-	)
-	(symbol
 		(lib_id "Device:Q_NPN_BEC")
 		(at 128.27 120.65 0)
@@
 			)
 		)
-		(property "Value" "56"
+		(property "Value" "1000"
 			(at 45.72 53.34 90)
 			(effects
@@
 			)
 		)
-		(property "Value" "56"
+		(property "Value" "10"
 			(at 115.57 73.66 90)
 			(effects
@@
 	)
 	(symbol
+		(lib_id "Device:Q_NPN_BEC")
+		(at 71.12 63.5 0)
+		(unit 1)
+		(exclude_from_sim no)
+		(in_bom yes)
+		(on_board yes)
+		(dnp no)
+		(fields_autoplaced yes)
+		(property "Reference" "Q8"
+			(at 76.2 62.2299 0)
+			(effects
+				(font
+					(size 1.27 1.27)
+				)
+				(justify left)
+			)
+		)
+		(property "Value" "Q_NPN_BEC"
+			(at 76.2 64.7699 0)
+			(effects
+				(font
+					(size 1.27 1.27)
+				)
+				(justify left)
+			)
+		)
+		(property "Footprint" "Package_TO_SOT_SMD:SOT-23-3"
+			(at 76.2 60.96 0)
+			(effects
+				(font
+					(size 1.27 1.27)
+				)
+				(hide yes)
+			)
+		)
+		(property "Datasheet" "~"
+			(at 71.12 63.5 0)
+			(effects
+				(font
+					(size 1.27 1.27)
+				)
+				(hide yes)
+			)
+		)
+		(property "Description" "NPN transistor, base/emitter/collector"
+			(at 71.12 63.5 0)
+			(effects
+				(font
+					(size 1.27 1.27)
+				)
+				(hide yes)
+			)
+		)
+		(pin "3"
+		)
+		(pin "1"
+		)
+		(pin "2"
+		)
+		(instances
+			(project "t41_2_power_amplifier"
+				(path "/2dfc3106-0fe9-4b2c-b32a-a54bf0a73e15"
+					(reference "Q8")
+					(unit 1)
+				)
+			)
+		)
+	)
+	(symbol
 		(lib_id "Device:Transformer_1P_1S")
 		(at 240.03 68.58 0)
@@
 			)
 		)
-		(property "Value" "56"
+		(property "Value" "150"
 			(at 99.06 73.66 90)
 			(effects

Commit message: Updated resistor values.
Parts:
- added L3: 10uH, Inductor_SMD:L_1210_3225Metric, symbol Device:L_Small
- R10, R4: value 1500 -> 270
- R12, R21: value 150 -> 100
- R13: value 10 -> 5
- R15, R16: value 56 -> 270
- R18: value 56 -> 20
- R3: value 1000 -> 1500
Connections:
- net 12V_IN_FIL: now also L3.1
- net at C15.2, Q7.3 (C), Q8.3 (C)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: now also L3.2
Changed lines of the file:
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@@
 	)
 	(junction
+		(at 73.66 39.37)
+		(diameter 0)
+		(color 0 0 0 0)
+	)
+	(junction
 		(at 175.26 82.55)
 		(diameter 0)
@@
 	)
 	(junction
+		(at 81.28 49.53)
+		(diameter 0)
+		(color 0 0 0 0)
+	)
+	(junction
 		(at 91.44 130.81)
 		(diameter 0)
@@
 	(wire
 		(pts
+			(xy 81.28 39.37) (xy 81.28 41.91)
+		)
+		(stroke
+			(width 0)
+			(type default)
+		)
+	)
+	(wire
+		(pts
 			(xy 71.12 144.78) (xy 73.66 144.78)
 		)
@@
 	(wire
 		(pts
+			(xy 81.28 46.99) (xy 81.28 49.53)
+		)
+		(stroke
+			(width 0)
+			(type default)
+		)
+	)
+	(wire
+		(pts
 			(xy 101.6 49.53) (xy 113.03 49.53)
 		)
@@
 	(wire
 		(pts
+			(xy 73.66 39.37) (xy 81.28 39.37)
+		)
+		(stroke
+			(width 0)
+			(type default)
+		)
+	)
+	(wire
+		(pts
 			(xy 100.33 172.72) (xy 100.33 175.26)
 		)
@@
 			)
 		)
-		(property "Value" "150"
+		(property "Value" "100"
 			(at 54.61 73.66 90)
 			(effects
@@
 			)
 		)
-		(property "Value" "56"
+		(property "Value" "20"
 			(at 35.56 60.96 90)
 			(effects
@@
 			)
 		)
-		(property "Value" "1500"
+		(property "Value" "270"
 			(at 90.17 73.66 90)
 			(effects
@@
 			)
 		)
-		(property "Value" "56"
+		(property "Value" "270"
 			(at 27.94 69.85 90)
 			(effects
@@
 			)
 		)
-		(property "Value" "1500"
+		(property "Value" "270"
 			(at 45.72 73.66 90)
 			(effects
@@
 			)
 		)
-		(property "Value" "1000"
+		(property "Value" "1500"
 			(at 45.72 53.34 90)
 			(effects
@@
 			)
 		)
-		(property "Value" "10"
+		(property "Value" "5"
 			(at 115.57 73.66 90)
 			(effects
@@
 	)
 	(symbol
+		(lib_id "Device:L_Small")
+		(at 81.28 44.45 0)
+		(unit 1)
+		(exclude_from_sim no)
+		(in_bom yes)
+		(on_board yes)
+		(dnp no)
+		(fields_autoplaced yes)
+		(property "Reference" "L3"
+			(at 82.55 43.1799 0)
+			(effects
+				(font
+					(size 1.27 1.27)
+				)
+				(justify left)
+			)
+		)
+		(property "Value" "10uH"
+			(at 82.55 45.7199 0)
+			(effects
+				(font
+					(size 1.27 1.27)
+				)
+				(justify left)
+			)
+		)
+		(property "Footprint" "Inductor_SMD:L_1210_3225Metric"
+			(at 81.28 44.45 0)
+			(effects
+				(font
+					(size 1.27 1.27)
+				)
+				(hide yes)
+			)
+		)
+		(property "Datasheet" "~"
+			(at 81.28 44.45 0)
+			(effects
+				(font
+					(size 1.27 1.27)
+				)
+				(hide yes)
+			)
+		)
+		(property "Description" "Inductor, small symbol"
+			(at 81.28 44.45 0)
+			(effects
+				(font
+					(size 1.27 1.27)
+				)
+				(hide yes)
+			)
+		)
+		(pin "2"
+		)
+		(pin "1"
+		)
+		(instances
+			(project "t41_2_power_amplifier"
+				(path "/2dfc3106-0fe9-4b2c-b32a-a54bf0a73e15"
+					(reference "L3")
+					(unit 1)
+				)
+			)
+		)
+	)
+	(symbol
 		(lib_id "Device:Q_PMOS_GSD")
 		(at 130.81 109.22 270)
@@
 			)
 		)
-		(property "Value" "56"
+		(property "Value" "270"
 			(at 38.1 69.85 90)
 			(effects
@@
 			)
 		)
-		(property "Value" "150"
+		(property "Value" "100"
 			(at 99.06 73.66 90)
 			(effects

Commit message: Clean-up prior to branch.
Parts:
- removed C21: 0.1uF, Capacitor_SMD:C_1206_3216Metric, symbol Device:C_Small
- removed E5: XXX, Inductor_SMD:L_1206_3216Metric, symbol 28F0121-0SR-10:28F0121-0SR-10
- removed L3: 10uH, Inductor_SMD:L_1210_3225Metric, symbol Device:L_Small
- removed Q5: Q_PMOS_GSD, Package_TO_SOT_SMD:SOT-23-3, symbol Device:Q_PMOS_GSD
- removed Q6: Q_NPN_BEC, Package_TO_SOT_SMD:SOT-23-3, symbol Device:Q_NPN_BEC
- removed R20: 10k, Resistor_SMD:R_1206_3216Metric, symbol Device:R_Small_US
- added C22, C23, C24: 0.1uF, Capacitor_SMD:C_1206_3216Metric, symbol Device:C_Small
- added C25, C26: 1uf, Capacitor_SMD:C_1206_3216Metric, symbol Device:C_Small
- added FB1: FerriteBead, symbol Device:FerriteBead
- added Q5: Q_NPN_BEC, Package_TO_SOT_SMD:SOT-23-3, symbol Device:Q_NPN_BEC
- added R20: 2k, Potentiometer_THT:Potentiometer_Bourns_3296W_Vertical, symbol Device:R_Potentiometer_US
- added R24, R25, R26: 10, Resistor_SMD:R_1206_3216Metric, symbol Device:R_Small_US
- added R27: 1.3k, Resistor_SMD:R_1206_3216Metric, symbol Device:R_Small_US
- added T1: Transformer_1P_SS, Binocular_Core:BN-43-302, symbol Device:Transformer_1P_SS
- added T5: Transformer_1P_SS, symbol Transformer_Double_Tapped:Transformer_1P_SS
- added U2: MCP1802x-xx02xOT, Package_TO_SOT_SMD:SOT-23-5, symbol Regulator_Linear:MCP1802x-xx02xOT
- added VR1: TL431AQDBZR_215, digikey-footprints:SOT-23-3, symbol dk_PMIC-Voltage-Reference:TL431AQDBZR_215
- C14: value 0.1uF -> 1.0uF
- Q2: footprint Package_TO_SOT_SMD:SOT-89-3 -> Package_TO_SOT_SMD:SOT-223
- R10: value 270 -> 810
- R12: value 100 -> 10
- R13: value 5 -> 10
- R19: value 10k -> 10
- R22: value 1000 -> 390
Connections:
- net 12V_IN_FIL: no longer R22.2
- net GND: now also C16.1, C4.1, C24.1, C25.2, C26.2, R20.3, R24.1, R25.1, R26.1, T5.5 (SC), U2.2 (GND), VR1.3 (A); no longer C4.2, R10.1, T3.1 (AA), T3.4 (SC)
- net TXRX: now also U2.3 (~{SHDN})
- net at Q7.3 (C), Q8.3 (C), R3.2: now also T1.1 (AA); no longer C15.2, R22.1
- net 12V_FIL: now reaches C10.1, C13.1, C20.1, C9.1, E1.1, E3.2, U1.1 (VIN)
- net 12V_FIL: now also C16.2, R19.1, C26.1, T5.2, U2.1 (VIN)
- net at T3.2 (AB): no longer C16.1
- net at L1.2, R14.1, R9.2: no longer C16.2, Q2.2 (C), Q4.4 (C)
- net 12V_PA: now reaches R19.2
- net 12V_PA: now also C1.1, E1.2, L2.2
- net at T3.3 (SA): no longer C6.2
- net at T3.5 (SB): no longer C5.2
- net at Q4.3 (E), R13.2: no longer Q4.1
- removed net 12V_OUT_FIL: C1.1, C4.1, E1.2, L2.2
- new net: Q5.2 (E), R12.2
- new net: R20.1, R22.1, R27.2, VR1.1 (K)
- new net: R20.2, VR1.2 (REF)
- new net: C24.2, FB1.1, T1.2 (AB)
- new net: Q4.2 (B), T1.3 (SA)
- new net: Q2.2 (B), T1.5 (SB)
- new net: Q2.3 (E), R24.2
- new net: Q4.1, R26.2
- new net: Q4.4 (C), T5.3 (AB)
- new net: Q2.1, R25.2
- new net: Q2.4 (C), T5.1 (AA)
- new net: C5.2, T5.6 (SB)
- new net: C6.2, T5.4 (SA)
- new net V12_REG: C25.1, FB1.2, R22.2, U2.5 (VOUT)
- new net Vmirror: C4.2, Q5.1 (B), Q5.3 (C), R27.1, T1.4 (SC)
- now unconnected: C15.1, R10.2, R9.1
Other:
- note added: "12V LOW DROP REGULATOR"
- note removed: "BFQ19 SOT-89"
- note removed: "P CHANNEL"
- moved on the sheet: C10, C11, C12, C13, C14, C15, C16, C17, C18, C19, C20, C5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
